Commit message: edit

File: src/fra333_lab2_25_v1/cocoa_description/robot/cocoa.urdf.xacro (robot description, xacro)
@@ -72,4 +72,5 @@
         <child link="link_3"/>
         <origin rpy="1.5708 0 0" xyz="0.0605 0 0.062"/>
+        <!-- <origin rpy="1.5708 0 0" xyz="0.0605 0 0"/> -->
         <axis xyz="0 0 1"/>
         <limit lower="0" upper="0.134" effort="0.5" velocity="0.5"/>

Commit message: edit

File: src/fra333_lab2_25_v1/cocoa_description/robot/cocoa.urdf.xacro (robot description, xacro)
@@ -71,6 +71,6 @@
         <parent link="link_2"/>
         <child link="link_3"/>
-        <origin rpy="1.5708 0 0" xyz="0.0605 0 0.062"/>
-        <!-- <origin rpy="1.5708 0 0" xyz="0.0605 0 0"/> -->
+        <origin rpy="1.5708 0 0" xyz="0.0605 -0.062 0"/>
+        <!-- <origin rpy="1.5708 0 0" xyz="0.0605 0 0.062"/> -->
         <axis xyz="0 0 1"/>
         <limit lower="0" upper="0.134" effort="0.5" velocity="0.5"/>

Commit message: edit

File: src/fra333_lab2_25_v1/cocoa_description/robot/cocoa.urdf.xacro (robot description, xacro)
@@ -88,5 +88,6 @@
         <parent link="link_3"/>
         <child link="end_effector"/>
-        <origin rpy="1.57 0 -1.57" xyz="-0.03 0 0.0282"/>
+        <!-- <origin rpy="1.57 0 -1.57" xyz="-0.03 0 0.0282"/> -->
+        <origin rpy="1.57 -1.57 1.57" xyz="-0.03 0 0.282"/>
         <axis xyz="0 0 1"/>
     </joint>

Commit message: edit

File: src/fra333_lab2_25_v1/cocoa_description/robot/cocoa.urdf.xacro (robot description, xacro)
@@ -33,5 +33,5 @@
             <mesh filename="package://cocoa_description/meshes/link_0.stl"/>
           </geometry>
-          <material name="Grey"/>
+          <material name="Orange"/>
         </visual>
       </link>
@@ -39,5 +39,5 @@
         <parent link="link_0"/>
         <child link="link_1"/>
-        <origin rpy="1.5708 0 1.5708" xyz="0 0 0"/>
+        <origin rpy="1.5708 0 0" xyz="0 0 0"/>
         <axis xyz="0 0 1"/>
         <limit lower="-0.523" upper="0.523" effort="0.5" velocity="0.5"/>
@@ -49,5 +49,5 @@
             <mesh filename="package://cocoa_description/meshes/link_1.stl"/>
           </geometry>
-          <material name="Grey"/>
+          <material name="Blue"/>
         </visual>
       </link>
@@ -55,5 +55,5 @@
         <parent link="link_1"/>
         <child link="link_2"/>
-        <origin rpy="0 0 0" xyz="0.262 0 0"/>
+        <origin rpy="0 0 1.5708" xyz="0 0.262 0"/>
         <axis xyz="0 0 1"/>
         <limit lower="-1.0472" upper="1.5708" effort="0.5" velocity="0.5"/>
@@ -65,5 +65,5 @@
             <mesh filename="package://cocoa_description/meshes/link_2.stl"/>
           </geometry>
-          <material name="Grey"/>
+          <material name="Orange"/>
         </visual>
       </link>
@@ -72,5 +72,4 @@
         <child link="link_3"/>
         <origin rpy="1.5708 0 0" xyz="0.0605 -0.062 0"/>
-        <!-- <origin rpy="1.5708 0 0" xyz="0.0605 0 0.062"/> -->
         <axis xyz="0 0 1"/>
         <limit lower="0" upper="0.134" effort="0.5" velocity="0.5"/>
@@ -82,5 +81,5 @@
             <mesh filename="package://cocoa_description/meshes/link_3.stl"/>
           </geometry>
-          <material name="Grey"/>
+          <material name="Blue"/>
         </visual>
       </link>
@@ -88,5 +87,4 @@
         <parent link="link_3"/>
         <child link="end_effector"/>
-        <!-- <origin rpy="1.57 0 -1.57" xyz="-0.03 0 0.0282"/> -->
         <origin rpy="1.57 -1.57 1.57" xyz="-0.03 0 0.282"/>
         <axis xyz="0 0 1"/>
@@ -98,5 +96,5 @@
             <mesh filename="package://cocoa_description/meshes/end_effector.stl"/>
           </geometry>
-          <material name="Grey"/>
+          <material name="Orange"/>
         </visual>
       </link>

Commit message: Edit l

File: src/fra333_lab2_25_v1/cocoa_description/robot/cocoa.urdf.xacro (robot description, xacro)
@@ -23,5 +23,5 @@
         <parent link="base_link"/>
         <child link="link_0"/>
-        <origin rpy="0 0 0" xyz="0 0 0.14"/>
+        <origin rpy="0 0 0" xyz="0 0 0.136"/>
         <axis xyz="0 0 1"/>
         <limit lower="-3.14" upper="3.14" effort="0.5" velocity="0.5"/>
@@ -87,5 +87,5 @@
         <parent link="link_3"/>
         <child link="end_effector"/>
-        <origin rpy="1.57 -1.57 1.57" xyz="-0.03 0 0.282"/>
+        <origin rpy="1.57 -1.57 1.57" xyz="-0.035 0 0.282"/>
         <axis xyz="0 0 1"/>
     </joint>

Commit message: IK done , no condition

File: src/fra333_lab2_25_v1/cocoa_description/robot/cocoa.urdf.xacro (robot description, xacro)
@@ -10,4 +10,7 @@
     <material name="Blue">
         <color rgba="0.5 0.7 1.0 1.0"/>
+    </material>
+    <material name="Red">
+      <color rgba="1.0 0.0 0.0 1.0"/>
     </material>
     <link name="base_link">
@@ -55,5 +58,5 @@
         <parent link="link_1"/>
         <child link="link_2"/>
-        <origin rpy="0 0 1.5708" xyz="0 0.262 0"/>
+        <origin rpy="0 0 0" xyz="0 0.262 0"/>
         <axis xyz="0 0 1"/>
         <limit lower="-1.0472" upper="1.5708" effort="0.5" velocity="0.5"/>
@@ -68,10 +71,10 @@
         </visual>
       </link>
-    <joint name="joint_pris_2_3" type="prismatic">
+    <joint name="joint_rev_2_3" type="revolute">
         <parent link="link_2"/>
         <child link="link_3"/>
-        <origin rpy="1.5708 0 0" xyz="0.0605 -0.062 0"/>
+        <origin rpy="0 0 0" xyz="0.18575 0 0"/>
         <axis xyz="0 0 1"/>
-        <limit lower="0" upper="0.134" effort="0.5" velocity="0.5"/>
+        <limit lower="-1.57" upper="0.523599" effort="0.5" velocity="0.5"/>
     </joint>
     <link name="link_3">
@@ -87,5 +90,5 @@
         <parent link="link_3"/>
         <child link="end_effector"/>
-        <origin rpy="1.57 -1.57 1.57" xyz="-0.035 0 0.282"/>
+        <origin rpy="-1.57 0 0" xyz="0.170 0 0"/>
         <axis xyz="0 0 1"/>
     </joint>
@@ -96,5 +99,5 @@
             <mesh filename="package://cocoa_description/meshes/end_effector.stl"/>
           </geometry>
-          <material name="Orange"/>
+          <material name="Red"/>
         </visual>
       </link>
