Commit message: update setting

File: src/fra333_lab3_25_v1/description/cocoa_gazebo.xacro (robot description, xacro)
@@ -90,5 +90,5 @@
         <material>Gazebo/Green</material>
     </gazebo>
-    <gazebo reference="link_2">
+    <!-- <gazebo reference="link_2">
         <mu1>0.2</mu1>
         <mu2>0.2</mu2>
@@ -99,5 +99,5 @@
         <mu2>0.2</mu2>
         <material>Gazebo/White</material>
-    </gazebo>
+    </gazebo> -->
     <!-- The next section shows an example of adding a sensor, in this case a depth camera. -->
     <!-- Due to a quirk of how cameras work, an extra joint/link is required to create an

File: src/fra333_lab3_25_v1/description/cocoa_include.xacro (robot description, xacro)
@@ -18,14 +18,15 @@
     <xacro:property name="link_0_c_offset_x" value="0.0"/>
     <xacro:property name="link_0_c_offset_y" value="0.0"/>
-    <xacro:property name="link_0_c_offset_z" value="0.0"/>
-    <xacro:property name="link_1_c_offset_x" value="0.0"/>
-    <xacro:property name="link_1_c_offset_y" value="0.0"/>
-    <xacro:property name="link_1_c_offset_z" value="0.0"/>
-    <xacro:property name="link_2_c_offset_x" value="0.0"/>
-    <xacro:property name="link_2_c_offset_y" value="0.0"/>
-    <xacro:property name="link_2_c_offset_z" value="0.0"/>
-    <xacro:property name="link_3_c_offset_x" value="0.0"/>
-    <xacro:property name="link_3_c_offset_y" value="0.0"/>
-    <xacro:property name="link_3_c_offset_z" value="0.0"/>
+    <xacro:property name="link_0_c_offset_z" value="0.009962"/>
+    <xacro:property name="link_1_c_offset_x" value="-0.027383"/>
+    <xacro:property name="link_1_c_offset_y" value="0.002656"/>
+    <xacro:property name="link_1_c_offset_z" value="-0.067605"/>
+    <!-- <xacro:property name="link_1_c_offset_z" value="1"/> -->
+    <xacro:property name="link_2_c_offset_x" value="-0.010935"/>
+    <xacro:property name="link_2_c_offset_y" value="0.099891"/>
+    <xacro:property name="link_2_c_offset_z" value="-0.003837"/>
+    <xacro:property name="link_3_c_offset_x" value="0.077878"/>
+    <xacro:property name="link_3_c_offset_y" value="0.054699"/>
+    <xacro:property name="link_3_c_offset_z" value="0.000125"/>
     <xacro:property name="end_c_offset_x" value="0.0"/>
     <xacro:property name="end_c_offset_y" value="0.0"/>

File: src/fra333_lab3_25_v1/description/cocoa_robot.urdf.xacro (robot description, xacro)
@@ -20,4 +20,5 @@
       <geometry>
         <mesh filename="file:///$(find fra333_lab3_25_v1)/meshes/link_0.stl"/>
+        <!-- <cylinder radius="0.21" length="0.020"/> -->
       </geometry>
       <material name="Grey"/>
@@ -25,14 +26,14 @@
     <collision>
         <origin xyz="${link_0_c_offset_x} ${link_0_c_offset_y} ${link_0_c_offset_z}" rpy="0 0 0"/>
-        <contact_coefficients mu="0" kp="1000.0" kd="1.0"/>
+        <contact_coefficients mu="0" kp="1.0" kd="1.0"/>
         <geometry>
             <mesh filename="file:///$(find fra333_lab3_25_v1)/meshes/link_0.stl"/>
-            <!-- <cylinder radius="1" length="0.5"/> -->
+            <!-- <cylinder radius="0.21" length="0.020"/> -->
         </geometry>
     </collision>
     <inertial>
-      <origin xyz="0 0 0.05" rpy="0 0 0"/>
-      <mass value="120" />
-      <inertia ixx="0" ixy="0.0" ixz="0.0" iyy="0" iyz="0.0" izz="0" />
+      <origin xyz="${link_0_c_offset_x} ${link_0_c_offset_y} ${link_0_c_offset_z}" rpy="0 0 0"/>
+      <mass value="0.689781" />
+      <inertia ixx="0.001916" ixy="0.000000" ixz="0.000000" iyy="0.001916" iyz="0.000000" izz="0.003787" />
     </inertial>
   </link>
@@ -54,5 +55,5 @@
     <collision>
         <origin xyz="${link_1_c_offset_x} ${link_1_c_offset_y} ${link_1_c_offset_z}" rpy="0 0 0"/>
-        <contact_coefficients mu="0" kp="1000.0" kd="1.0"/>
+        <contact_coefficients mu="0" kp="1.0" kd="1.0"/>
         <geometry>
             <mesh filename="file:///$(find fra333_lab3_25_v1)/meshes/link_1.stl"/>
@@ -61,7 +62,7 @@
     </collision>
     <inertial>
-      <origin xyz="0 0 0.05" rpy="0 0 0"/>
-      <mass value="120" />
-      <inertia ixx="0" ixy="0.0" ixz="0.0" iyy="0" iyz="0.0" izz="0" />
+      <origin xyz="${link_1_c_offset_x} ${link_1_c_offset_y} ${link_1_c_offset_z}" rpy="0 0 0"/>
+      <mass value="3.584649" />
+      <inertia ixx="0.012069" ixy="0.000340" ixz="0.000161" iyy="0.018044" iyz="0.000626" izz="0.024030" />
     </inertial>
   </link>
@@ -75,5 +76,5 @@
   <link name="link_2">
     <visual>
-      <origin rpy="${link_2_c_offset_x} ${link_2_c_offset_y} ${link_2_c_offset_z}" xyz="0 0 0"/>
+      <origin xyz="0 0 0.0" rpy="0 0 0"/>
       <geometry>
         <mesh filename="file:///$(find fra333_lab3_25_v1)/meshes/link_2.stl"/>
@@ -82,6 +83,6 @@
     </visual>
     <collision>
-        <origin xyz="0 0 0.0" rpy="0 0 0"/>
-        <contact_coefficients mu="0" kp="1000.0" kd="1.0"/>
+        <origin rpy="0 0 0" xyz="${link_2_c_offset_x} ${link_2_c_offset_y} ${link_2_c_offset_z}"/>
+        <contact_coefficients mu="0" kp="1.0" kd="1.0"/>
         <geometry>
             <mesh filename="file:///$(find fra333_lab3_25_v1)/meshes/link_2.stl"/>
@@ -90,7 +91,7 @@
     </collision>
     <inertial>
-      <origin xyz="0 0 0.05" rpy="0 0 0"/>
-      <mass value="120" />
-      <inertia ixx="0" ixy="0.0" ixz="0.0" iyy="0" iyz="0.0" izz="0" />
+      <origin rpy="0 0 0" xyz="${link_2_c_offset_x} ${link_2_c_offset_y} ${link_2_c_offset_z}"/>
+      <mass value="1.674836" />
+      <inertia ixx="0.012791" ixy="0.000469" ixz="-0.000258" iyy="0.002594" iyz="0.000898" izz="0.012890" />
     </inertial>
   </link>
@@ -104,5 +105,5 @@
   <link name="link_3">
     <visual>
-      <origin rpy="${link_3_c_offset_x} ${link_3_c_offset_y} ${link_3_c_offset_z}" xyz="0 0 0"/>
+      <origin xyz="0 0 0" rpy="0 0 0"/>
       <geometry>
         <mesh filename="file:///$(find fra333_lab3_25_v1)/meshes/link_3.stl"/>
@@ -111,6 +112,6 @@
     </visual>
     <collision>
-        <origin xyz="0 0 0.0" rpy="0 0 0"/>
-        <contact_coefficients mu="0" kp="1000.0" kd="1.0"/>
+        <origin rpy="0 0 0" xyz="${link_3_c_offset_x} ${link_3_c_offset_y} ${link_3_c_offset_z}"/>
+        <contact_coefficients mu="0" kp="1.0" kd="1.0"/>
         <geometry>
             <mesh filename="file:///$(find fra333_lab3_25_v1)/meshes/link_3.stl"/>
@@ -119,7 +120,7 @@
     </collision>
     <inertial>
-      <origin xyz="0 0 0.05" rpy="0 0 0"/>
-      <mass value="120" />
-      <inertia ixx="0" ixy="0.0" ixz="0.0" iyy="0" iyz="0.0" izz="0" />
+      <origin rpy="0 0 0" xyz="${link_3_c_offset_x} ${link_3_c_offset_y} ${link_3_c_offset_z}"/>
+      <mass value="1.783530" />
+      <inertia ixx="0.002620" ixy="-0.000433" ixz="0.000004" iyy="0.010684" iyz="-0.000003" izz="0.011479" />
     </inertial>
   </link>

Commit message: add param

File: src/fra333_lab3_25_v1/description/cocoa_gazebo.xacro (robot description, xacro)
@@ -90,5 +90,5 @@
         <material>Gazebo/Green</material>
     </gazebo>
-    <!-- <gazebo reference="link_2">
+    <gazebo reference="link_2">
         <mu1>0.2</mu1>
         <mu2>0.2</mu2>
@@ -98,6 +98,6 @@
         <mu1>0.2</mu1>
         <mu2>0.2</mu2>
-        <material>Gazebo/White</material>
-    </gazebo> -->
+        <material>Gazebo/Green</material>
+    </gazebo>
     <!-- The next section shows an example of adding a sensor, in this case a depth camera. -->
     <!-- Due to a quirk of how cameras work, an extra joint/link is required to create an

File: src/fra333_lab3_25_v1/description/cocoa_include.xacro (robot description, xacro)
@@ -22,10 +22,9 @@
     <xacro:property name="link_1_c_offset_y" value="0.002656"/>
     <xacro:property name="link_1_c_offset_z" value="-0.067605"/>
-    <!-- <xacro:property name="link_1_c_offset_z" value="1"/> -->
-    <xacro:property name="link_2_c_offset_x" value="-0.010935"/>
-    <xacro:property name="link_2_c_offset_y" value="0.099891"/>
+    <xacro:property name="link_2_c_offset_x" value="0.099891"/>
+    <xacro:property name="link_2_c_offset_y" value="0.010935"/>
     <xacro:property name="link_2_c_offset_z" value="-0.003837"/>
-    <xacro:property name="link_3_c_offset_x" value="0.077878"/>
-    <xacro:property name="link_3_c_offset_y" value="0.054699"/>
+    <xacro:property name="link_3_c_offset_x" value="0.054699"/>
+    <xacro:property name="link_3_c_offset_y" value="-0.077878"/>
     <xacro:property name="link_3_c_offset_z" value="0.000125"/>
     <xacro:property name="end_c_offset_x" value="0.0"/>

File: src/fra333_lab3_25_v1/description/cocoa_robot.urdf.xacro (robot description, xacro)
@@ -17,5 +17,5 @@
   <link name="link_0">
     <visual>
-      <origin rpy="0 0 0" xyz="0 0 0"/>
+      <origin xyz="0 0 0" rpy="0 0 0"/>
       <geometry>
         <mesh filename="file:///$(find fra333_lab3_25_v1)/meshes/link_0.stl"/>
@@ -25,5 +25,5 @@
     </visual>
     <collision>
-        <origin xyz="${link_0_c_offset_x} ${link_0_c_offset_y} ${link_0_c_offset_z}" rpy="0 0 0"/>
+        <origin xyz="0 0 0" rpy="0 0 0"/>
         <contact_coefficients mu="0" kp="1.0" kd="1.0"/>
         <geometry>
@@ -47,5 +47,5 @@
   <link name="link_1">
     <visual>
-      <origin rpy="0 0 0" xyz="0 0 0"/>
+      <origin xyz="0 0 0" rpy="0 0 0"/>
       <geometry>
         <mesh filename="file:///$(find fra333_lab3_25_v1)/meshes/link_1.stl"/>
@@ -54,10 +54,10 @@
     </visual>
     <collision>
-        <origin xyz="${link_1_c_offset_x} ${link_1_c_offset_y} ${link_1_c_offset_z}" rpy="0 0 0"/>
-        <contact_coefficients mu="0" kp="1.0" kd="1.0"/>
-        <geometry>
-            <mesh filename="file:///$(find fra333_lab3_25_v1)/meshes/link_1.stl"/>
-            <!-- <box size="2.5 1.5 0.1" /> -->
-        </geometry>
+      <origin xyz="0 0 0" rpy="0 0 0"/>
+      <contact_coefficients mu="0" kp="1.0" kd="1.0"/>
+      <geometry>
+          <mesh filename="file:///$(find fra333_lab3_25_v1)/meshes/link_1.stl"/>
+          <!-- <box size="2.5 1.5 0.1" /> -->
+      </geometry>
     </collision>
     <inertial>
@@ -70,5 +70,5 @@
     <parent link="link_1"/>
     <child link="link_2"/>
-    <origin rpy="1.5708 0 0" xyz="0 0 0"/>
+    <origin rpy="1.5708 -1.5708 0" xyz="0 0 0"/>
     <axis xyz="0 0 1"/>
     <limit lower="-0.523" upper="0.523" effort="0.5" velocity="0.5"/>
@@ -83,15 +83,15 @@
     </visual>
     <collision>
-        <origin rpy="0 0 0" xyz="${link_2_c_offset_x} ${link_2_c_offset_y} ${link_2_c_offset_z}"/>
-        <contact_coefficients mu="0" kp="1.0" kd="1.0"/>
-        <geometry>
-            <mesh filename="file:///$(find fra333_lab3_25_v1)/meshes/link_2.stl"/>
-            <!-- <box size="2.5 1.5 0.1" /> -->
-        </geometry>
+      <origin xyz="0 0 0" rpy="0 0 0"/>
+      <contact_coefficients mu="0" kp="1.0" kd="1.0"/>
+      <geometry>
+          <mesh filename="file:///$(find fra333_lab3_25_v1)/meshes/link_2.stl"/>
+          <!-- <box size="2.5 1.5 0.1" /> -->
+      </geometry>
     </collision>
     <inertial>
-      <origin rpy="0 0 0" xyz="${link_2_c_offset_x} ${link_2_c_offset_y} ${link_2_c_offset_z}"/>
+      <origin xyz="${link_2_c_offset_x} ${link_2_c_offset_y} ${link_2_c_offset_z}" rpy="0 0 0"/>
       <mass value="1.674836" />
-      <inertia ixx="0.012791" ixy="0.000469" ixz="-0.000258" iyy="0.002594" iyz="0.000898" izz="0.012890" />
+      <inertia ixx="0.002594" ixy="-0.000469" ixz="0.000898" iyy="0.012791" iyz="0.000258" izz="0.012890" />
     </inertial>
   </link>
@@ -99,5 +99,5 @@
     <parent link="link_2"/>
     <child link="link_3"/>
-    <origin rpy="0 0 0" xyz="0 0.261 0"/>
+    <origin rpy="0 0 0" xyz="0.261 0 0"/>
     <axis xyz="0 0 1"/>
     <limit lower="-1.0472" upper="1.5708" effort="0.5" velocity="0.5"/>
@@ -112,24 +112,16 @@
     </visual>
     <collision>
-        <origin rpy="0 0 0" xyz="${link_3_c_offset_x} ${link_3_c_offset_y} ${link_3_c_offset_z}"/>
-        <contact_coefficients mu="0" kp="1.0" kd="1.0"/>
-        <geometry>
-            <mesh filename="file:///$(find fra333_lab3_25_v1)/meshes/link_3.stl"/>
-            <!-- <box size="2.5 1.5 0.1" /> -->
-        </geometry>
+      <origin xyz="0 0 0" rpy="0 0 0"/>
+      <contact_coefficients mu="0" kp="1.0" kd="1.0"/>
+      <geometry>
+          <mesh filename="file:///$(find fra333_lab3_25_v1)/meshes/link_3.stl"/>
+          <!-- <box size="2.5 1.5 0.1" /> -->
+      </geometry>
     </collision>
     <inertial>
-      <origin rpy="0 0 0" xyz="${link_3_c_offset_x} ${link_3_c_offset_y} ${link_3_c_offset_z}"/>
+      <origin xyz="${link_3_c_offset_x} ${link_3_c_offset_y} ${link_3_c_offset_z}" rpy="0 0 0"/>
       <mass value="1.783530" />
-      <inertia ixx="0.002620" ixy="-0.000433" ixz="0.000004" iyy="0.010684" iyz="-0.000003" izz="0.011479" />
+      <inertia ixx="0.010684" ixy="0.000433" ixz="-0.000003" iyy="0.002620" iyz="-0.000004" izz="0.011479" />
     </inertial>
-  </link>
-  <joint name="joint_eff" type="fixed">
-    <parent link="link_3"/>
-    <child link="end_effector"/>
-    <origin rpy="-1.57 0 0" xyz="0.170 0 0"/>
-    <axis xyz="0 0 1"/>
-  </joint>
-  <link name="end_effector">
   </link>
   <xacro:include filename="cocoa_gazebo.xacro" />
