Commit message: urdf done

File: src/fra333_lab3_25_v1/description/cocoa_gazebo.xacro (robot description, xacro)
@@ -1,146 +1,97 @@
 <?xml version="1.0"?>
 <robot xmlns:xacro="http://www.ros.org/wiki/xacro">
-    <!-- This file demonstrates the use of some <gazebo> tags -->
-    <!-- To include it add the following line -->
-    <!-- <xacro:include filename="example_gazebo.xacro" /> -->
-    <!-- Gazebo is unable to use the same <material> tags that are already in the URDF (that RViz uses). -->
-    <!-- Instead, we need to add gazebo tags for our links that refer to Gazebo materials -->
-    <!-- <gazebo reference="slider_link">
-        <material>Gazebo/Blue</material>
-    </gazebo>
-    <gazebo reference="arm_link">
-        <material>Gazebo/Orange</material>
-    </gazebo> -->
-    <!-- Gazebo requires the use of plugins to interact with other systems such as ROS. -->
-    <!-- This plugin will publish the joint_states for the selected joints
-            (which robot_state_publisher can then use to broadcast the approprate tf). -->
-    <!-- <gazebo>
-        <plugin name="gazebo_ros_joint_state_publisher"
-            filename="libgazebo_ros_joint_state_publisher.so">
-            <update_rate>20</update_rate>
-            <joint_name>joint_1</joint_name>
-            <joint_name>joint_2</joint_name>
-            <joint_name>joint_3</joint_name>
-        </plugin>
-    </gazebo> -->
-    <!-- This plugin will read a JointTrajectory message from the /set_joint_trajectory topic
-            and move the machine accordingly. It's a bit clunky but it works. -->
-    <!-- You'll probably want to add damping to the joints to stop them it flopping around.
-            e.g. <dynamics damping="10.0" friction="10.0"/> -->
-    <!-- Here's an example message to publish to test it:
-            ros2 topic pub -1 /set_joint_trajectory trajectory_msgs/msg/JointTrajectory  '{header: {frame_id: world}, joint_names: [slider_joint, arm_joint], points: [  {positions: {0.8,0.6}} ]}' -->
-    <gazebo>
-        <plugin name="gazebo_ros_joint_pose_trajectory"
-            filename="libgazebo_ros_joint_pose_trajectory.so">
-            <update_rate>2</update_rate>
-        </plugin>
-    </gazebo>
-    <ros2_control name="GazeboSystem" type="system">
-        <hardware>
-          <plugin>gazebo_ros2_control/GazeboSystem</plugin>
-        </hardware>
-        <joint name="joint_rev_0_1">
-            <command_interface name="position">
-                <param name="min">-3.14</param>
-                <param name="max">3.14</param>
-            </command_interface>
-            <state_interface name="position">
-                <param name="initial_value">0.0</param>
-            </state_interface>
-            <state_interface name="velocity"/>
-            <state_interface name="effort"/>
-        </joint>
-        <joint name="joint_rev_1_2">
-            <command_interface name="position">
-                <param name="min">-3.14</param>
-                <param name="max">3.14</param>
-            </command_interface>
-            <state_interface name="position">
-                <param name="initial_value">0.0</param>
-            </state_interface>
-            <state_interface name="velocity"/>
-            <state_interface name="effort"/>
-        </joint>
-        <joint name="joint_rev_2_3">
-            <command_interface name="position">
-                <param name="min">-3.14</param>
-                <param name="max">3.14</param>
-            </command_interface>
-            <state_interface name="position">
-                <param name="initial_value">0.0</param>
-            </state_interface>
-            <state_interface name="velocity"/>
-            <state_interface name="effort"/>
-        </joint>
-      </ros2_control>
-    <gazebo>
-        <plugin filename="libgazebo_ros2_control.so" name="gazebo_ros2_control">
-            <robot_sim_type>gazebo_ros2_control/GazeboSystem</robot_sim_type>
-          <parameters>$(find fra333_lab3_25_v1)/config/myrobot_controllers.yaml</parameters>
-        </plugin>
-    </gazebo>
-    <gazebo reference="link_0">
-        <mu1>0.2</mu1>
-        <mu2>0.2</mu2>
-        <material>Gazebo/Red</material>
-    </gazebo>
-    <gazebo reference="link_1">
-        <mu1>0.2</mu1>
-        <mu2>0.2</mu2>
-        <material>Gazebo/Green</material>
-    </gazebo>
-    <gazebo reference="link_2">
-        <mu1>0.2</mu1>
-        <mu2>0.2</mu2>
-        <material>Gazebo/Black</material>
-    </gazebo>
-    <gazebo reference="link_3">
-        <mu1>0.2</mu1>
-        <mu2>0.2</mu2>
-        <material>Gazebo/Green</material>
-    </gazebo>
-    <!-- The next section shows an example of adding a sensor, in this case a depth camera. -->
-    <!-- Due to a quirk of how cameras work, an extra joint/link is required to create an
-            "optical frame" for the sensor. That isn't the focus for this tutorial, but you can
-            look at https://www.ros.org/reps/rep-0103.html#suffix-frames for slightly more information. -->
-    <!-- First, create the link and joint for the optical frame -->
-    <!-- <joint name="camera_optical_joint" type="fixed">
-        <origin xyz="0 0 0" rpy="-1.571 0 -1.571" />
-        <parent link="camera_link" />
-        <child link="camera_link_optical" />
+  <gazebo>
+    <plugin name="gazebo_ros_joint_pose_trajectory"
+      filename="libgazebo_ros_joint_pose_trajectory.so">
+      <update_rate>2</update_rate>
+    </plugin>
+  </gazebo>
+  <ros2_control name="GazeboSystem" type="system">
+    <hardware>
+      <plugin>gazebo_ros2_control/GazeboSystem</plugin>
+    </hardware>
+    <joint name="joint_rev_0_1">
+      <command_interface name="position">
+          <param name="min">-3.14</param>
+          <param name="max">3.14</param>
+      </command_interface>
+      <command_interface name="velocity">
+        <param name="min">-10</param>
+        <param name="max">10</param>
+      </command_interface>
+      <command_interface name="effort">
+        <param name="min">-1000</param>
+        <param name="max">1000</param>
+      </command_interface>
+      <state_interface name="position">
+          <param name="initial_value">0.0</param>
+      </state_interface>
+      <state_interface name="velocity"/>
+      <state_interface name="effort"/>
     </joint>
-    <link name="camera_link_optical"></link> -->
-    <!-- Add a gazebo tag for the ORIGINAL camera_link (but in the plugin we reference the optical frame so that ROS can orient things correctly) -->
-    <!-- Within the gazebo tag we have the sensor tag, and inside that there is (among other things) the camera tag with the camera parameters,
-            and the plugin tag with some extra parameters the plugin needs. -->
-    <!-- Note that although visualise is set to true, it won't actually visualise the depth camera in gazebo. To see the preview,
-            try swapping "depth" to "camera"-->
-    <!-- <gazebo reference="camera_link">
-        <sensor type="depth" name="my_camera">
-            <update_rate>20</update_rate>
-            <visualize>true</visualize>
-            <camera name="cam">
-                <horizontal_fov>1.3962634</horizontal_fov>
-                <image>
-                    <width>640</width>
-                    <height>480</height>
-                    <format>R8B8G8</format>
-                </image>
-                <clip>
-                    <near>0.02</near>
-                    <far>300</far>
-                </clip>
-                <noise>
-                    <type>gaussian</type>
-                    <mean>0.0</mean>
-                    <stddev>0.007</stddev>
-                </noise>
-            </camera>
-            <plugin name="camera_controller" filename="libgazebo_ros_camera.so">
-                <frame_name>camera_link_optical</frame_name>
-                <min_depth>0.1</min_depth>
-                <max_depth>500</max_depth>
-            </plugin>
-        </sensor>
-    </gazebo> -->
+    <joint name="joint_rev_1_2">
+      <command_interface name="position">
+          <param name="min">-3.14</param>
+          <param name="max">3.14</param>
+      </command_interface>
+      <command_interface name="velocity">
+        <param name="min">-10</param>
+        <param name="max">10</param>
+      </command_interface>
+      <command_interface name="effort">
+        <param name="min">-1000</param>
+        <param name="max">1000</param>
+      </command_interface>
+      <state_interface name="position">
+          <param name="initial_value">0.0</param>
+      </state_interface>
+      <state_interface name="velocity"/>
+      <state_interface name="effort"/>
+    </joint>
+    <joint name="joint_rev_2_3">
+      <command_interface name="position">
+          <param name="min">-3.14</param>
+          <param name="max">3.14</param>
+      </command_interface>
+      <command_interface name="velocity">
+        <param name="min">-10</param>
+        <param name="max">10</param>
+      </command_interface>
+      <command_interface name="effort">
+        <param name="min">-1000</param>
+        <param name="max">1000</param>
+      </command_interface>
+      <state_interface name="position">
+          <param name="initial_value">0.0</param>
+      </state_interface>
+      <state_interface name="velocity"/>
+      <state_interface name="effort"/>
+    </joint>
+  </ros2_control>
+  <gazebo>
+      <plugin filename="libgazebo_ros2_control.so" name="gazebo_ros2_control">
+          <robot_sim_type>gazebo_ros2_control/GazeboSystem</robot_sim_type>
+        <parameters>$(find fra333_lab3_25_v1)/config/cocoa_controllers.yaml</parameters>
+      </plugin>
+  </gazebo>
+  <gazebo reference="link_0">
+      <mu1>0.2</mu1>
+      <mu2>0.2</mu2>
+      <material>Gazebo/Red</material>
+  </gazebo>
+  <gazebo reference="link_1">
+      <mu1>0.2</mu1>
+      <mu2>0.2</mu2>
+      <material>Gazebo/Green</material>
+  </gazebo>
+  <gazebo reference="link_2">
+      <mu1>0.2</mu1>
+      <mu2>0.2</mu2>
+      <material>Gazebo/Black</material>
+  </gazebo>
+  <gazebo reference="link_3">
+      <mu1>0.2</mu1>
+      <mu2>0.2</mu2>
+      <material>Gazebo/Blue</material>
+  </gazebo>
 </robot>

File: src/fra333_lab3_25_v1/description/cocoa_include.xacro (robot description, xacro)
@@ -28,7 +28,4 @@
     <xacro:property name="link_3_c_offset_y" value="-0.077878"/>
     <xacro:property name="link_3_c_offset_z" value="0.000125"/>
-    <xacro:property name="end_c_offset_x" value="0.0"/>
-    <xacro:property name="end_c_offset_y" value="0.0"/>
-    <xacro:property name="end_c_offset_z" value="0.0"/>
     <!-- Specify some standard inertial calculations https://en.wikipedia.org/wiki/List_of_moments_of_inertia -->
     <!-- These make use of xacro's mathematical functionality -->

File: src/fra333_lab3_25_v1/description/cocoa_robot.urdf.xacro (robot description, xacro)
@@ -6,4 +6,5 @@
   <!-- This will include all the contents of example_include.xacro first. Go check it out! -->
   <xacro:include filename="cocoa_include.xacro" />
+  <xacro:include filename="cocoa_gazebo.xacro" />
   <!-- This first link called "world" is empty -->
   <link name="world"></link>
@@ -20,5 +21,4 @@
       <geometry>
         <mesh filename="file:///$(find fra333_lab3_25_v1)/meshes/link_0.stl"/>
-        <!-- <cylinder radius="0.21" length="0.020"/> -->
       </geometry>
       <material name="Grey"/>
@@ -26,8 +26,7 @@
     <collision>
         <origin xyz="0 0 0" rpy="0 0 0"/>
-        <contact_coefficients mu="0" kp="1.0" kd="1.0"/>
+        <contact_coefficients mu="0" kp="1000.0" kd="1.0"/>
         <geometry>
             <mesh filename="file:///$(find fra333_lab3_25_v1)/meshes/link_0.stl"/>
-            <!-- <cylinder radius="0.21" length="0.020"/> -->
         </geometry>
     </collision>
@@ -43,5 +42,5 @@
     <origin rpy="0 0 0" xyz="0 0 0.136"/>
     <axis xyz="0 0 1"/>
-    <limit lower="-3.14" upper="3.14" effort="0.5" velocity="0.5"/>
+    <limit lower="-3.14" upper="3.14" effort="1.0" velocity="1.0"/>
   </joint>
   <link name="link_1">
@@ -55,8 +54,7 @@
     <collision>
       <origin xyz="0 0 0" rpy="0 0 0"/>
-      <contact_coefficients mu="0" kp="1.0" kd="1.0"/>
+      <contact_coefficients mu="0" kp="1000.0" kd="1.0"/>
       <geometry>
           <mesh filename="file:///$(find fra333_lab3_25_v1)/meshes/link_1.stl"/>
-          <!-- <box size="2.5 1.5 0.1" /> -->
       </geometry>
     </collision>
@@ -72,5 +70,5 @@
     <origin rpy="1.5708 -1.5708 0" xyz="0 0 0"/>
     <axis xyz="0 0 1"/>
-    <limit lower="-0.523" upper="0.523" effort="0.5" velocity="0.5"/>
+    <limit lower="-0.523" upper="0.523" effort="1.0" velocity="1.0"/>
   </joint>
   <link name="link_2">
@@ -84,8 +82,7 @@
     <collision>
       <origin xyz="0 0 0" rpy="0 0 0"/>
-      <contact_coefficients mu="0" kp="1.0" kd="1.0"/>
+      <contact_coefficients mu="0" kp="1000.0" kd="1.0"/>
       <geometry>
           <mesh filename="file:///$(find fra333_lab3_25_v1)/meshes/link_2.stl"/>
-          <!-- <box size="2.5 1.5 0.1" /> -->
       </geometry>
     </collision>
@@ -99,7 +96,7 @@
     <parent link="link_2"/>
     <child link="link_3"/>
-    <origin rpy="0 0 0" xyz="0.261 0 0"/>
+    <origin rpy="0 0 0" xyz="0.26179 0 0"/>
     <axis xyz="0 0 1"/>
-    <limit lower="-1.0472" upper="1.5708" effort="0.5" velocity="0.5"/>
+    <limit lower="-1.0472" upper="1.5708" effort="1.0" velocity="1.0"/>
   </joint>
   <link name="link_3">
@@ -113,8 +110,7 @@
     <collision>
       <origin xyz="0 0 0" rpy="0 0 0"/>
-      <contact_coefficients mu="0" kp="1.0" kd="1.0"/>
+      <contact_coefficients mu="0" kp="1000.0" kd="1.0"/>
       <geometry>
           <mesh filename="file:///$(find fra333_lab3_25_v1)/meshes/link_3.stl"/>
-          <!-- <box size="2.5 1.5 0.1" /> -->
       </geometry>
     </collision>
@@ -125,4 +121,18 @@
     </inertial>
   </link>
-  <xacro:include filename="cocoa_gazebo.xacro" />
+  <joint name="joint_eff" type="fixed">
+    <parent link="link_3"/>
+    <child link="end_effector"/>
+    <origin rpy="-1.5708 0 -1.5708" xyz="0 -0.200 0"/>
+    <axis xyz="0 0 1"/>
+  </joint>
+  <link name="end_effector">
+    <visual>
+      <origin xyz="0 0 0" rpy="0 0 0"/>
+      <geometry>
+        <mesh filename="file:///$(find fra333_lab3_25_v1)/meshes/end_effector.stl"/>
+      </geometry>
+      <material name="Blue"/>
+    </visual>
+  </link>
 </robot>

File: src/fra333_lab3_25_v1/description/example_gazebo.xacro (robot description, xacro)
@@ -88,5 +88,5 @@
         <mu1>0.2</mu1>
         <mu2>0.2</mu2>
-        <material>Gazebo/Green</material>
+        <material>Gazebo/Orange</material>
     </gazebo>
     <gazebo reference="link_2">
@@ -98,5 +98,5 @@
         <mu1>0.2</mu1>
         <mu2>0.2</mu2>
-        <material>Gazebo/Black</material>
+        <material>Gazebo/Blue</material>
     </gazebo>
     <!-- The next section shows an example of adding a sensor, in this case a depth camera. -->

File: src/fra333_lab3_25_v1/description/test.urdf.xacro (robot description, xacro)
@@ -31,7 +31,14 @@
     <parent link="link_3"/>
     <child link="end_effector"/>
-    <origin rpy="0 0 0" xyz="0.170 0 0"/>
+    <origin rpy="0 0 0" xyz="0 -0.120 0"/>
     <axis xyz="0 0 1"/>
   </joint>
   <link name="end_effector">
+    <visual>
+      <origin xyz="0 0 0" rpy="0 0 0"/>
+      <geometry>
+        <mesh filename="file:///$(find fra333_lab3_25_v1)/meshes/end_effector.stl"/>
+      </geometry>
+      <material name="Blue"/>
+    </visual>
   </link>

File: src/ros2_control_demo_3r_robot/description/example_gazebo.xacro (robot description, xacro)
@@ -74,10 +74,10 @@
         </joint>
       </ros2_control>
-    <!-- <gazebo>
+    <gazebo>
         <plugin filename="libgazebo_ros2_control.so" name="gazebo_ros2_control">
             <robot_sim_type>gazebo_ros2_control/GazeboSystem</robot_sim_type>
           <parameters>$(find ros2_control_demo_3r_robot)/config/myrobot_controllers.yaml</parameters>
         </plugin>
-    </gazebo> -->
+    </gazebo>
     <gazebo reference="link0">
         <mu1>0.2</mu1>
