Commit message: done v2

File: src/fra333_lab3_25_v1/cocoav_description/robot/cocoav_robot.urdf.xacro (robot description, xacro)
@@ -42,5 +42,5 @@
     <origin rpy="0 0 0" xyz="0 0 0.136"/>
     <axis xyz="0 0 1"/>
-    <limit lower="-3.14" upper="3.14" effort="1.0" velocity="1.0"/>
+    <limit lower="-6.28" upper="6.28" effort="1.0" velocity="1.0"/>
   </joint>
   <link name="link_1">
