Commit message: update new version

File: src/fra333_lab4_25_v1/cocoax_description/robot/cocoax_include.xacro (robot description, xacro)
@@ -15,4 +15,13 @@
     <material name="Red">
     <color rgba="1.0 0.0 0.0 1.0"/>
+    </material>
+    <material name="Black">
+        <color rgba="0.0 0.0 0.0 0.6"/>
+    </material>
+    <material name="White">
+        <color rgba="1.0 1.0 1.0 1.0"/>
+    </material>
+    <material name="DarkBlue">
+        <color rgba="0.0 0.0 0.3764 0.6"/>
     </material>
     <xacro:property name="link_0_c_offset_x" value="0.0"/>

File: src/fra333_lab4_25_v1/cocoax_description/robot/cocoax_robot.urdf.xacro (robot description, xacro)
@@ -50,5 +50,5 @@
         <mesh filename="file:///$(find cocoax_description)/meshes/link_1.stl"/>
       </geometry>
-      <material name="Orange"/>
+      <material name="White"/>
     </visual>
     <collision>
@@ -124,5 +124,5 @@
     <parent link="link_3"/>
     <child link="end_effector"/>
-    <origin rpy="-1.5708 0 -1.5708" xyz="0 -0.200 0"/>
+    <origin rpy="-1.5708 0 -1.5708" xyz="0 -0.245 0"/>
     <axis xyz="0 0 1"/>
   </joint>
@@ -133,5 +133,5 @@
         <mesh filename="file:///$(find cocoax_description)/meshes/end_effector.stl"/>
       </geometry>
-      <material name="Blue"/>
+      <material name="White"/>
     </visual>
   </link>
